File: Hardware/SparkFun_Capacitive_Soil_Moisture_Sensor.kicad_pcb (KiCad board)
At the start: 2 copper layers, 15.2 x 76.2 mm, 57 parts, among them J1 Qwiic_RA, J2 Qwiic_RA, U1 CY8CMBR3102

Commit message: Roll version for reds and increase silk font
Parts:
- removed kibuzzard-693B4BBA (x2): G***, kibuzzard-693B4BBA
- removed kibuzzard-693B4BC8 (x2): G***, kibuzzard-693B4BC8
- removed kibuzzard-693B4BFF (x2): G***, kibuzzard-693B4BFF
- removed kibuzzard-693B4C16 (x2): G***, kibuzzard-693B4C16
- removed kibuzzard-693B4C27 (x2): G***, kibuzzard-693B4C27
- removed kibuzzard-693B4C3E (x2): G***, kibuzzard-693B4C3E
- removed kibuzzard-693B4C4C: G***, kibuzzard-693B4C4C
- removed kibuzzard-693B4C5A: G***, kibuzzard-693B4C5A
- added kibuzzard-6969377A: G***, kibuzzard-6969377A, F.Cu at (115.6, 74.9)
- added kibuzzard-69693786: G***, kibuzzard-69693786, B.Cu at (115.6, 74.9)
- added kibuzzard-6969378A: G***, kibuzzard-6969378A, F.Cu at (113.3, 80.0)
- added kibuzzard-69693792: G***, kibuzzard-69693792, F.Cu at (113.3, 86.4)
- added kibuzzard-69693797: G***, kibuzzard-69693797, F.Cu at (113.3, 92.7)
- added kibuzzard-6969379D: G***, kibuzzard-6969379D, F.Cu at (113.3, 99.1)
- added kibuzzard-696937A1: G***, kibuzzard-696937A1, F.Cu at (113.3, 105.4)
- added kibuzzard-696937A5: G***, kibuzzard-696937A5, F.Cu at (113.3, 111.8)
- added kibuzzard-696937B5: G***, kibuzzard-696937B5, B.Cu at (117.8, 86.4)
- added kibuzzard-696937B9: G***, kibuzzard-696937B9, B.Cu at (117.8, 92.7)
- added kibuzzard-696937BE: G***, kibuzzard-696937BE, B.Cu at (117.8, 99.1)
- added kibuzzard-696937C3: G***, kibuzzard-696937C3, B.Cu at (117.8, 105.4)
- added kibuzzard-696937C9: G***, kibuzzard-696937C9, B.Cu at (117.8, 111.8)
- added kibuzzard-696937DE: G***, kibuzzard-696937DE, B.Cu at (117.8, 80.0)
Other:
- board text added: "v10"
- board text removed: "v01"
